File: pcb/dongle/dongle.kicad_pcb (KiCad board)
At the start: 2 copper layers, 143.2 x 85.8 mm, 35 parts, among them J1 Bat, M1 MOUNT, M2 MOUNT, M3 MOUNT, M4 MOUNT, M5 MOUNT, M6 MOUNT, M7 MOUNT, M8 MOUNT, SW1 SW_Reset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

Commit message: Battery connections added
Routing:
- net GND: track 38.3 -> 39.0 mm
Other:
- rule pad_to_mask_clearance: 0.038 -> 0
